File: Hardware/32U4_Breakout.sch (EAGLE design)
At the start: 33 parts, among them J1 AVR_SPI_PRG, U1 ATMEGA32U4, U2 3.3V_REG_LDOSMD, X1 USBSMD, Y1 16MHz

Commit message: Updated to v12 eagle files
Eagle files for QC board revision and schematic updates.
Parts:
- removed JP4: LOGO-SFENEW, SparkFun:LOGO-SFENEW
- removed JP5: LOGO-SFESK, SparkFun:LOGO-SFESK
- removed TP1, TP2: TEST-POINT3, SparkFun:TEST-POINT3
- removed U$7: CREATIVE_COMMONS, SparkFun:CREATIVE_COMMONS
- added JP8: LOGO-SFENEW, SparkFun-Aesthetics:LOGO-SFENEW
- C1, C2, C3, C4, C5, C6, C7, C9: device SparkFun:CAP0402-CAP -> SparkFun-Capacitors:CAP0603-CAP
- JP6, JP7: value FIDUCIALUFIDUCIAL -> FIDUCIAL1X2; device SparkFun:FIDUCIALUFIDUCIAL -> SparkFun:FIDUCIAL1X2
- R1, R2, R3, R4: device SparkFun:RESISTOR0402-RES -> SparkFun-Resistors:RESISTOR0603-RES
- U1: device SparkFun:ATMEGA32U4QFN2 -> Testing:ATMEGA32U41:1
Connections:
- net D+: no longer TP1.1
- net D-: no longer TP2.1
Other:
- note added: "-all vias now .015"
- note added: "-bottom silk labels for all pins"
- note added: "-changed CAP and RES packages to be 0603, routed as necessary"
- note added: "-revised footprint of IC to be 1:1, adjusted routes as necessary"
- note added: "-shifted ic and isp headers each one grid space to the right."
- note added: "5V by default"
- note added: "Changes for v12:"
- note added: "Revised by: Kade Jensen"
- note added: "v12"
- note removed: "v11"
