File: Production Files/32U4_Breakout-Panel-v12.brd (EAGLE design)
At the start: 142.7 x 116.8 mm, 363 parts, among them J1 AVR_SPI_PRG, J10 AVR_SPI_PRG, J11 AVR_SPI_PRG, J12 AVR_SPI_PRG, J2 AVR_SPI_PRG, J3 AVR_SPI_PRG, J4 AVR_SPI_PRG, J5 AVR_SPI_PRG, J6 AVR_SPI_PRG, J7 AVR_SPI_PRG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

Commit message: changed paste layer on IC
Parts:
- U1, U11, U13, U15, U17, U19, U21, U23, U3, U5, U7, U9: device Testing:QFN-44-NOPAD_1:1 -> Testing:QFN-44-NOPAD_1:1-LESS_PASTE
